File: elec/layout/default/stm32h723vg.kicad_pcb (KiCad board)
At the start: 2 copper layers, 225.7 x 100.8 mm, 0 parts

Commit message: dev board layout complete
Parts:
- added C1: 6.3V 2.2uF X5R ±20% 0402 Multilayer Ceramic Capacitors MLCC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, lib:C0402, F.Cu at (213.4, 42.2)
- added C10: 16V 100nF X7R ±10% 0402 Multilayer Ceramic Capacitors MLCC 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, lib:C0402, F.Cu at (215.8, 53.7)
- added C11: 16V 100nF X7R ±10% 0402 Multilayer Ceramic Capacitors MLCC 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, lib:C0402, F.Cu at (207.3, 46.2)
- added C12: 16V 100nF X7R ±10% 0402 Multilayer Ceramic Capacitors MLCC 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, lib:C0402, F.Cu at (207.3, 47.2)
- added C13: 25V 1uF X5R ±10% 0402 Multilayer Ceramic Capacitors MLCC - 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, lib:C0402, F.Cu at (207.3, 50.8)
- added C14: 16V 100nF X7R ±10% 0402 Multilayer Ceramic Capacitors MLCC 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, lib:C0402, F.Cu at (213.8, 52.7)
- added C15: 25V 1uF X5R ±10% 0402 Multilayer Ceramic Capacitors MLCC - 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, lib:C0402, F.Cu at (213.8, 53.7)
- added C16: 16V 100nF X7R ±10% 0402 Multilayer Ceramic Capacitors MLCC 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, lib:C0402, F.Cu at (207.2, 49.3)
- added C2: 6.3V 2.2uF X5R ±20% 0402 Multilayer Ceramic Capacitors MLCC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, lib:C0402, F.Cu at (212.4, 42.2)
- added C3: 10V 4.7uF X5R ±20% 0402 Multilayer Ceramic Capacitors MLCC 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, lib:C0402, F.Cu at (207.3, 45.2)
- added C4: 16V 100nF X7R ±10% 0402 Multilayer Ceramic Capacitors MLCC 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, lib:C0402, F.Cu at (217.8, 51.5)
- added C5: 16V 100nF X7R ±10% 0402 Multilayer Ceramic Capacitors MLCC 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, lib:C0402, F.Cu at (207.2, 44.2)
- added C6: 16V 100nF X7R ±10% 0402 Multilayer Ceramic Capacitors MLCC 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, lib:C0402, F.Cu at (215.8, 52.7)
- added C7: 16V 100nF X7R ±10% 0402 Multilayer Ceramic Capacitors MLCC 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, lib:C0402, F.Cu at (217.8, 52.6)
- added C8: 16V 100nF X7R ±10% 0402 Multilayer Ceramic Capacitors MLCC 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, lib:C0402, F.Cu at (217.8, 53.7)
- added C9: 16V 100nF X7R ±10% 0402 Multilayer Ceramic Capacitors MLCC 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, lib:C0402, F.Cu at (207.3, 48.3)
- added R1: 62.5mW Thick Film Resistors 50V ±100ppm/℃ ±1% 10kΩ 0402 Chi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, lib:R0402, F.Cu at (224.0, 45.6)
- added U1: , lib:TFBGA-100_L8.0-W8.0-R10-C10-P0.80-BL, F.Cu at (212.6, 47.9)
- added U2: , lib:KEY-SMD_4P-L4.2-W3.2-P2.20-LS4.6, F.Cu at (221.7, 47.2)
Routing:
- net boot0: track 0.00 -> 1.53 mm
